File: project source/ESP32-S3_Audio_Control_Board/Audio.kicad_sch (KiCad schematic)
At the start: 1 part, among them U4 TAS5805MPWP

Commit message: update
Parts:
- added C25: 4.7u, Capacitor_SMD:C_0603_1608Metric, symbol Device:C
- added C26: 100n, Capacitor_SMD:C_0402_1005Metric, symbol Device:C
- added C27, C29: 390uF, Capacitor_SMD:CP_Elec_8x10.5, symbol Device:CP
- added C28, C30: 22u, Capacitor_SMD:C_1206_3216Metric, symbol Device:C
- added C31, C32: 100n, Capacitor_SMD:C_0603_1608Metric, symbol Device:C
- added C33, C35: 220n, Capacitor_SMD:C_0603_1608Metric, symbol Device:C
- added C34, C36: 680n, Capacitor_SMD:C_1206_3216Metric, symbol Device:C
- added C37, C38: 1u, Capacitor_SMD:C_0402_1005Metric, symbol Device:C
- added H1, H2, H3, H4: MountingHole, MountingHole:MountingHole_3.2mm_M3_Pad_Via, symbol Mechanical:MountingHole
- added L3, L4: 10u, Inductor_SMD:L_KOHERelec_MDA7030, symbol pspice:INDUCTOR
- added R18: 10K, Resistor_SMD:R_0402_1005Metric, symbol Device:R
- added R19: 4.7K, Resistor_SMD:R_0402_1005Metric, symbol Device:R
Connections:
- net DOUT: now also U4.8 (SDIN)
- net GND: now also C25.2, C26.2, C27.2, C28.2, C29.2, C30.2, C31.2, C32.2, C34.1, C36.1, C37.2, C38.2
- net PDN: now reaches U4.12 (~{PDN})
- net PDN: now also R18.2
- net at U4.13 (AVDD): now also C38.1
- net 12V: now reaches U4.15 (PVDD), U4.16 (PVDD), U4.27 (PVDD), U4.28 (PVDD)
- net 12V: now also C27.1, C28.1, C29.1, C30.1, C31.1, C32.1
- net 3V3: now reaches U4.2 (DVDD)
- net 3V3: now also C25.1, C26.1, R18.1, R19.1
- net at U4.22 (BST_A-): now also C35.1
- net at U4.23 (OUT_A-): now also C35.2, L4.1
- net at U4.25 (BST_A+): now also C33.1
- net at U4.26 (OUT_A+): now also C33.2, L3.1
- net ADR_FAULT: now reaches U4.3 (ADR/~{FAULT})
- net ADR_FAULT: now also R19.2
- net at U4.4 (VR_DIG): now also C37.1
- new net SPK_N: C36.2, L4.2
- new net SPK_P: C34.2, L3.2
- no-connect marks 0 -> 5
Other:
- note added: "I2C Address: 0x58"
- moved on the sheet: U4
