File: project source/ESP32-S3_Audio_Control_Board/ESP32-S3.kicad_sch (KiCad schematic)
At the start: 6 parts, among them SW3 SMD_4.6x2.8mm_h2.5mm, U1 ESP32-S3-WROOM-1

Commit message: update
Parts:
- added C3, C4, C6: 100n, Capacitor_SMD:C_0402_1005Metric, symbol Device:C
- added R1, R3: 1K, Resistor_SMD:R_0402_1005Metric, symbol Device:R
- added R4: 10K, Resistor_SMD:R_0402_1005Metric, symbol Device:R
- added R5, R6: 4.7K, Resistor_SMD:R_0402_1005Metric, symbol Device:R
- added TP1, TP2, TP3, TP4, TP5, TP6, TP7: IO0, TestPoint:TestPoint_Pad_D1.5mm, symbol Connector:TestPoint
- SW1: renamed from SW3; value SMD_4.6x2.8mm_h2.5mm -> SMD Buuton; footprint SparkFun-Switch:Momentary_SMD_4.6x2.8mm_h2.5mm -> Button_Switch_SMD:SW_SPST_EVQP2_MiddlePushTravel_H2.5mm; Mfr (none) -> ALPSALPINE; Mfr PN (none) -> SKRPABE010; PROD_ID SWCH-15606 -> (none); Part Description (none) -> -30℃~+85℃ 1.6N 100,000 cycles 16V 2.5mm 3.2mm 4.2mm 50mA J-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; Supplier (none) -> LCSC; Supplier PN (none) -> C115360
- renumbered C9 to C1, C10 to C2, C8 to C5, R37 to R2
Connections:
- net GND: now also C3.2, C4.2, C6.2, TP3.1
- net USB_DM: now reaches U1.13 (USB_D-)
- net USB_DP: now reaches U1.14 (USB_D+)
- net PDM_CLK: now reaches U1.17 (IO9)
- net PDM_DATA: now reaches U1.19 (IO11)
- net ADR_FAULT: now reaches U1.22 (IO14)
- net PDN: now reaches U1.23 (IO21)
- net SDA: now reaches U1.24 (IO47)
- net SDA: now also R6.2
- net SCL: now reaches U1.25 (IO48)
- net SCL: now also R5.2
- net IO0: now reaches U1.27 (IO0)
- net IO0: now also R4.2, TP6.1, TP7.1
- net WS_LED_DATA: now reaches U1.31 (IO38)
- net RXD: now reaches U1.36 (RXD0)
- net TXD: now reaches U1.37 (TXD0)
- net ADC1_CH1: now reaches U1.38 (IO2)
- net ADC1_CH1: now also C6.1, R3.2
- net ADC1_CH0: now reaches U1.39 (IO1)
- net ADC1_CH0: now also C4.1, R1.2
- net BTN: now reaches U1.4 (IO4)
- net COB_LED_DATA: now reaches U1.5 (IO5)
- net 3.3V renamed 3V3
- net 3V3: now also C3.1, R4.1, R5.1, R6.1, TP1.1
- new net EN: TP5.1
- new net POT1_ADC: R1.1
- new net POT2_ADC: R3.1
- new net RX: TP4.1
- new net TX: TP2.1
- no-connect marks 0 -> 3
Other:
- note added: "1: SPI BOOT 0: USB/UART BOOT"
- note added: "UART"
- moved on the sheet: C2, C5, R2, SW1
