File: project source/ESP32-S3_Audio_Control_Board/ESP32-S3_Audio_Control_Board.kicad_pcb (KiCad board)
At the start: 2 copper layers, 36 parts, among them J19 Barrel_Jack, Q1 DMP3013SFV-7, U1 ESP32-S3-WROOM-1, U2 TPS54331D, U4 TAS5805MPWP, U5 SN74AHCT1G125DBVR, U6 TPS54331D

Commit message: update
Parts:
- removed L5, L6: 6.8u, Inductor_SMD:L_Bourns_SRP7028A_7.3x6.6mm
- added C1: 22u, Capacitor_SMD:C_0603_1608Metric, B.Cu at (52.6, 153.9)
- added C11: 47u, Capacitor_SMD:C_1210_3225Metric, F.Cu at (38.0, 176.5)
- added C12: 47u, Capacitor_SMD:C_1210_3225Metric, F.Cu at (34.7, 176.5)
- added C15: 1n, Capacitor_SMD:C_0402_1005Metric, F.Cu at (19.4, 175.0)
- added C16: 47p, Capacitor_SMD:C_0402_1005Metric, F.Cu at (21.4, 175.0)
- added C2: 4.7u, Capacitor_SMD:C_0402_1005Metric, B.Cu at (58.4, 154.1)
- added C21: 47u, Capacitor_SMD:C_1210_3225Metric, F.Cu at (39.4, 158.5)
- added C22: 47u, Capacitor_SMD:C_1210_3225Metric, F.Cu at (36.1, 158.5)
- added C23: 1n, Capacitor_SMD:C_0402_1005Metric, F.Cu at (19.8, 161.2)
- added C24: 47p, Capacitor_SMD:C_0402_1005Metric, F.Cu at (22.0, 161.2)
- added C25: 4.7u, Capacitor_SMD:C_0603_1608Metric, F.Cu at (102.2, 170.8)
- added C26: 100n, Capacitor_SMD:C_0402_1005Metric, F.Cu at (102.2, 173.4)
- added C27: 390uF, Capacitor_SMD:CP_Elec_8x10.5, F.Cu at (89.6, 174.3)
- added C28: 22u, Capacitor_SMD:C_1206_3216Metric, B.Cu at (112.3, 158.5)
- added C29: 390uF, Capacitor_SMD:CP_Elec_8x10.5, F.Cu at (89.7, 185.4)
- added C3: 100n, Capacitor_SMD:C_0402_1005Metric, B.Cu at (55.8, 153.9)
- added C30: 22u, Capacitor_SMD:C_1206_3216Metric, B.Cu at (99.1, 158.8)
- added C31: 100n, Capacitor_SMD:C_0603_1608Metric, F.Cu at (110.4, 171.4)
- added C32: 100n, Capacitor_SMD:C_0603_1608Metric, F.Cu at (110.7, 177.6)
- added C33: 220n, Capacitor_SMD:C_0603_1608Metric, F.Cu at (109.5, 163.5)
- added C34: 680n, Capacitor_SMD:C_1206_3216Metric, F.Cu at (108.7, 183.0)
- added C35: 220n, Capacitor_SMD:C_0603_1608Metric, F.Cu at (106.5, 163.5)
- added C36: 680n, Capacitor_SMD:C_1206_3216Metric, F.Cu at (108.7, 190.0)
- added C37: 1u, Capacitor_SMD:C_0402_1005Metric, F.Cu at (107.6, 154.0)
- added C38: 1u, Capacitor_SMD:C_0402_1005Metric, F.Cu at (101.9, 154.0)
- added C39: 100n, Capacitor_SMD:C_0402_1005Metric, F.Cu at (47.4, 140.4)
- added C4: 100n, Capacitor_SMD:C_0402_1005Metric, B.Cu at (75.9, 163.2)
- added C40.1: 100n, Capacitor_SMD:C_0402_1005Metric, F.Cu at (59.0, 210.4)
- added C5: 1u, Capacitor_SMD:C_0402_1005Metric, B.Cu at (63.3, 152.7)
- added C6: 100n, Capacitor_SMD:C_0402_1005Metric, B.Cu at (75.9, 158.2)
- added D2: MMBZ5242BLT3G, Package_TO_SOT_SMD:TSOT-23, F.Cu at (14.5, 148.1)
- added F1: Fuse 3A, Resistor_SMD:R_1812_4532Metric, F.Cu at (22.9, 148.5)
- added H1: MountingHole, MountingHole:MountingHole_3.2mm_M3_Pad_Via, F.Cu at (17.2, 142.8)
- added H2: MountingHole, MountingHole:MountingHole_3.2mm_M3_Pad_Via, F.Cu at (17.2, 192.8)
- added H3: MountingHole, MountingHole:MountingHole_3.2mm_M3_Pad_Via, F.Cu at (67.2, 192.8)
- added H4: MountingHole, MountingHole:MountingHole_3.2mm_M3_Pad_Via, F.Cu at (67.2, 142.8)
- added J2: Conn_01x05_Pin, Connector_JST:JST_PH_B5B-PH-K_1x05_P2.00mm_Vertical, F.Cu at (52.7, 140.0)
- added J3: Conn_01x03_Pin, Connector_JST:JST_PH_B3B-PH-K_1x03_P2.00mm_Vertical, F.Cu at (40.5, 140.0)
- added J4: Conn_01x04_Pin, Connector_JST:JST_PH_B4B-PH-K_1x04_P2.00mm_Vertical, F.Cu at (54.7, 195.5)
- added J5: Conn_01x03_Pin, Connector_JST:JST_PH_B3B-PH-K_1x03_P2.00mm_Vertical, F.Cu at (31.5, 195.5)
- added J6: Conn_01x02_Pin, Connector_JST:JST_PH_B2B-PH-K_1x02_P2.00mm_Vertical, F.Cu at (14.5, 186.1)
- added L1: 6.8u, Inductor_SMD:L_Sunlord_MWSA0602S, F.Cu at (29.5, 168.7)
- added L2: 6.8u, Inductor_SMD:L_Sunlord_MWSA0602S, F.Cu at (28.5, 161.4)
- added L3: 10u, Inductor_SMD:L_KOHERelec_MDA7030, F.Cu at (121.5, 153.7)
- added L4: 10u, Inductor_SMD:L_KOHERelec_MDA7030, F.Cu at (121.5, 161.8)
- added R1: 1K, Resistor_SMD:R_0402_1005Metric, B.Cu at (75.9, 162.2)
- added R18: 10K, Resistor_SMD:R_0402_1005Metric, F.Cu at (104.2, 153.5)
- added R19: 4.7K, Resistor_SMD:R_0402_1005Metric, F.Cu at (109.6, 153.5)
- added R2: 10K, Resistor_SMD:R_0402_1005Metric, B.Cu at (63.4, 151.0)
- added R20: 100Ω, Resistor_SMD:R_0402_1005Metric, F.Cu at (49.6, 146.4)
- added R21: 100Ω, Resistor_SMD:R_0402_1005Metric, F.Cu at (56.1, 210.4)
- added R3: 1K, Resistor_SMD:R_0402_1005Metric, B.Cu at (75.9, 157.2)
- added R4: 10K, Resistor_SMD:R_0402_1005Metric, B.Cu at (49.5, 172.0)
- added R5: 4.7K, Resistor_SMD:R_0402_1005Metric, B.Cu at (49.5, 170.8)
- added R6: 4.7K, Resistor_SMD:R_0402_1005Metric, B.Cu at (49.5, 169.6)
- added TP1: IO0, TestPoint:TestPoint_Pad_D1.5mm, B.Cu at (99.5, 129.8)
- added TP10: IO0, TestPoint:TestPoint_Pad_D1.5mm, B.Cu at (91.9, 137.0)
- added TP2: IO0, TestPoint:TestPoint_Pad_D1.5mm, B.Cu at (96.5, 129.8)
- added TP4: IO0, TestPoint:TestPoint_Pad_D1.5mm, B.Cu at (96.5, 133.3)
- added TP5: IO0, TestPoint:TestPoint_Pad_D1.5mm, B.Cu at (99.5, 136.8)
- added TP6: IO0, TestPoint:TestPoint_Pad_D1.5mm, B.Cu at (96.5, 136.8)
- added TP7: IO0, TestPoint:TestPoint_Pad_D1.5mm, B.Cu at (91.8, 141.5)
- added TP8: IO0, TestPoint:TestPoint_Pad_D1.5mm, B.Cu at (91.9, 129.9)
- added TP9: IO0, TestPoint:TestPoint_Pad_D1.5mm, B.Cu at (91.9, 133.4)
- added U3: TPS54331D, Package_SO:SOIC-8-1EP_3.9x4.9mm_P1.27mm_EP2.29x3mm, F.Cu at (19.7, 157.8)
- C13: renamed from C36; moved to B.Cu
- C14: renamed from C40; moved to B.Cu
- Q1: value DMP3013SFV-7 -> AO3401A; footprint Package_SON:Diodes_PowerDI3333-8 -> Package_TO_SOT_SMD:SOT-23
- R10: renamed from R26; moved to B.Cu
- TP3: value TestPoint -> IO0; footprint TestPoint:TestPoint_Pad_2.0x2.0mm -> TestPoint:TestPoint_Pad_D1.5mm; moved to B.Cu
- U2: footprint Audio_control_board:TPS54331 -> Package_SO:SOIC-8-1EP_3.9x4.9mm_P1.27mm_EP2.29x3mm
- U6: value TPS54331D -> SN74AHCT1G125DBVR; footprint Audio_control_board:TPS54331 -> Audio_control_board:SOT95P280X145-5N__SN74AHCT1G125
- moved U5 147.9 mm to (46.5, 145.2), turned to 90 degrees
- moved U2 123.0 mm to (19.4, 171.5)
- moved C7 107.1 mm to (15.3, 167.3), turned to 90 degrees
- moved C8 107.1 mm to (13.3, 167.2), turned to 90 degrees
- moved C18 103.2 mm to (13.7, 156.1), turned to 90 degrees
- moved U6 102.4 mm to (52.1, 210.4)
- moved C17 100.6 mm to (16.3, 153.6)
- moved C41 100.5 mm to (17.0, 150.9)
- moved U4 99.4 mm to (105.7, 158.6), turned to -90 degrees
- moved C42 94.3 mm to (15.6, 174.9), turned to 90 degrees
- moved R13 94.0 mm to (14.2, 159.3), turned to 90 degrees
- moved C9 93.7 mm to (15.0, 170.4), turned to 90 degrees
- moved R7 93.7 mm to (14.0, 172.6), turned to 90 degrees
- moved Q1 92.6 mm to (19.0, 148.1)
- moved R15 92.6 mm to (15.4, 159.3), turned to -90 degrees
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- renumbered C46 to C10, C52 to C17, C54 to C18, C55 to C19, C53 to C20, C42 to C41, C45 to C42, C51 to C43, C41 to C7, C43 to C8, C44 to C9, D2 to D1, J19 to J1, R29 to R11, R30 to R12, R32 to R13, R35 to R14, R33 to R15, R34 to R16, R36 to R17, R27 to R7, R31 to R8, R28 to R9
Connections:
- C13 pad 1: Net-(Q1-D) -> Net-(C13-Pad1)
- C14 pad 2: Net-(D4-A) -> Net-(D2-A)
- C20 pad 1: Net-(U6-BOOT) -> Net-(U3-BOOT)
- C43 pad 2: Net-(U6-SS) -> Net-(U3-SS)
- J1 pad 1: Net-(Q1-D) -> Net-(C13-Pad1)
- Q1 pad 1: 12V -> Net-(D2-A)
- Q1 pad 3: 12V -> Net-(Q1-D)
- R10 pad 1: Net-(D4-A) -> Net-(D2-A)
- R13 pad 2: Net-(U6-EN) -> Net-(U3-EN)
- R14 pad 2: Net-(U6-VSENSE) -> Net-(U3-VSENSE)
- R15 pad 1: Net-(U6-EN) -> Net-(U3-EN)
- R17 pad 1: Net-(U6-VSENSE) -> Net-(U3-VSENSE)
- R8 pad 1: 3.3V -> 3V3
- TP3 pad 1: 12V -> GND
- U1 pad 13: unconnected-(U1-USB_D--Pad13) -> USB_DM
- U1 pad 14: unconnected-(U1-USB_D+-Pad14) -> USB_DP
- U1 pad 17: unconnected-(U1-IO9-Pad17) -> PDM_CLK
- U1 pad 19: unconnected-(U1-IO11-Pad19) -> PDM_DATA
- U1 pad 2: 3.3V -> 3V3
- U1 pad 22: unconnected-(U1-IO14-Pad22) -> ADR_FAULT
- U1 pad 23: unconnected-(U1-IO21-Pad23) -> PDN
- U1 pad 24: unconnected-(U1-IO47-Pad24) -> SDA
- U1 pad 25: unconnected-(U1-IO48-Pad25) -> SCL
- U1 pad 27: unconnected-(U1-IO0-Pad27) -> /ESP32-S3/IO0
- U1 pad 31: unconnected-(U1-IO38-Pad31) -> WS_LED_DATA
- U1 pad 36: unconnected-(U1-RXD0-Pad36) -> /ESP32-S3/RXD
- U1 pad 37: unconnected-(U1-TXD0-Pad37) -> /ESP32-S3/TXD
- U1 pad 38: unconnected-(U1-IO2-Pad38) -> /ESP32-S3/ADC1_CH1
- U1 pad 39: unconnected-(U1-IO1-Pad39) -> /ESP32-S3/ADC1_CH0
- U1 pad 4: unconnected-(U1-IO4-Pad4) -> BTN
- U1 pad 5: unconnected-(U1-IO5-Pad5) -> COB_LED_DATA
- U4 pad 12: unconnected-(U4-~{PDN}-Pad12) -> PDN
- U4 pad 13: unconnected-(U4-AVDD-Pad13) -> Net-(U4-AVDD)
- U4 pad 15: Net-(U4-PVDD-Pad15) -> 12V
- U4 pad 16: Net-(U4-PVDD-Pad15) -> 12V
- U4 pad 2: unconnected-(U4-DVDD-Pad2) -> 3V3
- U4 pad 22: unconnected-(U4-BST_A--Pad22) -> Net-(U4-BST_A-)
- U4 pad 23: unconnected-(U4-OUT_A--Pad23) -> Net-(U4-OUT_A-)
- U4 pad 25: unconnected-(U4-BST_A+-Pad25) -> Net-(U4-BST_A+)
- U4 pad 26: unconnected-(U4-OUT_A+-Pad26) -> Net-(U4-OUT_A+)
- U4 pad 27: Net-(U4-PVDD-Pad15) -> 12V
- U4 pad 28: Net-(U4-PVDD-Pad15) -> 12V
- U4 pad 3: unconnected-(U4-ADR/~{FAULT}-Pad3) -> ADR_FAULT
- U4 pad 4: unconnected-(U4-VR_DIG-Pad4) -> Net-(U4-VR_DIG)
- U4 pad 8: unconnected-(U4-SDIN-Pad8) -> DOUT
- U5 pad 1: unconnected-(U5-~{OE}-Pad1) -> GND
- U5 pad 2: unconnected-(U5-A-Pad2) -> Net-(U5-A)
- U5 pad 4: unconnected-(U5-Y-Pad4) -> /Peripheral/COB_LED
- U5 pad 5: unconnected-(U5-VCC-Pad5) -> 5V
- U6 pad 1: Net-(U6-BOOT) -> GND
- U6 pad 2: 12V -> Net-(U6-A)
- U6 pad 3: Net-(U6-EN) -> GND
- U6 pad 4: Net-(U6-SS) -> /Peripheral/WS_LED
- U6 pad 5: Net-(U6-VSENSE) -> 5V
Other:
- board outline added: 60 x 60 mm
