File: project source/ESP32-S3_Audio_Control_Board/ESP32-S3_Audio_Control_Board.kicad_sch (KiCad schematic)
At the start: 0 parts

Commit message: update
Other:
- sheet Power ports: added 5V; removed none
- note added: "ESP32-S3-WROOM-1-N16R8"
- note added: "LED"
- note added: "SN74AHCT1G125"
- note added: "TAS5805M"
- note added: "TPS54331"
Changed lines of the file:
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@@
 	(generator_version "10.0")
 	(paper "A4")
+	(text "ESP32-S3-WROOM-1-N16R8"
+		(exclude_from_sim no)
+		(at 74.93 71.882 0)
+		(effects
+			(font
+				(size 2.54 2.54)
+				(thickness 0.3175)
+			)
+		)
+	)
+	(text "SN74AHCT1G125"
+		(exclude_from_sim no)
+		(at 220.218 77.47 0)
+		(effects
+			(font
+				(size 2.54 2.54)
+				(thickness 0.3175)
+			)
+		)
+	)
+	(text "TAS5805M"
+		(exclude_from_sim no)
+		(at 146.558 116.332 0)
+		(effects
+			(font
+				(size 2.54 2.54)
+				(thickness 0.3175)
+			)
+		)
+	)
+	(text "LED"
+		(exclude_from_sim no)
+		(at 219.456 71.628 0)
+		(effects
+			(font
+				(size 2.54 2.54)
+				(thickness 0.3175)
+			)
+		)
+	)
+	(text "TPS54331"
+		(exclude_from_sim no)
+		(at 146.05 72.39 0)
+		(effects
+			(font
+				(size 2.54 2.54)
+				(thickness 0.3175)
+			)
+		)
+	)
+	(wire
+		(pts
+			(xy 177.8 67.31) (xy 189.23 67.31)
+		)
+		(stroke
+			(width 0)
+			(type default)
+		)
+	)
+	(label "5V"
+		(at 181.61 67.31 0)
+		(effects
+			(font
+				(size 1.27 1.27)
+			)
+			(justify left bottom)
+		)
+	)
 	(sheet
 		(at 116.84 55.88)
@@
 				)
 				(justify left top)
+			)
+		)
+		(pin "5V" output
+			(at 177.8 67.31 0)
+			(effects
+				(font
+					(size 1.27 1.27)
+				)
+				(justify right)
 			)
 		)
@@
 	)
 	(sheet
-		(at 116.84 101.6)
+		(at 116.84 100.33)
 		(size 60.96 30.48)
 		(exclude_from_sim no)
@@
 		)
 		(property "Sheetname" "Audio"
-			(at 116.84 100.8884 0)
+			(at 116.84 99.6184 0)
 			(show_name no)
 			(do_not_autoplace no)
@@
 		)
 		(property "Sheetfile" "Audio.kicad_sch"
-			(at 116.84 132.6646 0)
+			(at 116.84 131.3946 0)
 			(show_name yes)
 			(do_not_autoplace no)
@@
 	)
 	(sheet
-		(at 43.18 55.88)
+		(at 44.45 55.88)
 		(size 60.96 30.48)
 		(exclude_from_sim no)
@@
 		)
 		(property "Sheetname" "ESP32-S3"
-			(at 43.18 55.1684 0)
+			(at 44.45 55.1684 0)
 			(show_name no)
 			(do_not_autoplace no)
@@
 		)
 		(property "Sheetfile" "ESP32-S3.kicad_sch"
-			(at 43.18 86.9446 0)
+			(at 44.45 86.9446 0)
 			(show_name yes)
 			(do_not_autoplace no)
@@
 	)
 	(sheet
-		(at 190.5 101.6)
+		(at 189.23 55.88)
 		(size 60.96 30.48)
 		(exclude_from_sim no)
@@
 		)
 		(property "Sheetname" "Peripheral"
-			(at 190.5 100.8884 0)
+			(at 189.23 55.1684 0)
 			(show_name no)
 			(do_not_autoplace no)
@@
 		)
 		(property "Sheetfile" "Peri.kicad_sch"
-			(at 190.5 132.6646 0)
-			(show_name yes)
-			(do_not_autoplace no)
+			(at 189.23 86.9446 0)
+			(show_name yes)
+			(do_not_autoplace no)
