File: project source/ESP32-S3_Audio_Control_Board/Peri.kicad_sch (KiCad schematic)
At the start: 1 part, among them U5 SN74AHCT1G125DBVR

Commit message: update
Parts:
- added C39, C40.1: 100n, Capacitor_SMD:C_0402_1005Metric, symbol Device:C
- added J2: Conn_01x05_Pin, Connector_JST:JST_PH_B5B-PH-K_1x05_P2.00mm_Vertical, symbol Connector:Conn_01x05_Pin
- added J3, J5: Conn_01x03_Pin, Connector_JST:JST_PH_B3B-PH-K_1x03_P2.00mm_Vertical, symbol Connector:Conn_01x03_Pin
- added J4: Conn_01x04_Pin, Connector_JST:JST_PH_B4B-PH-K_1x04_P2.00mm_Vertical, symbol Connector:Conn_01x04_Pin
- added J6: Conn_01x02_Pin, Connector_JST:JST_PH_B2B-PH-K_1x02_P2.00mm_Vertical, symbol Connector:Conn_01x02_Pin
- added R20, R21: 100Ω, Resistor_SMD:R_0402_1005Metric, symbol Device:R
- added U6: SN74AHCT1G125DBVR, Audio_control_board:SOT95P280X145-5N__SN74AHCT1G125, symbol SN74AHCT1G125:SN74AHCT1G125DBVR
Connections:
- net GND: now also U5.1 (~{OE}), C39.2, C40.1.2, J2.2 (Pin_2), J3.1 (Pin_1), J4.1 (Pin_1), J5.1 (Pin_1), U6.1 (~{OE}), U6.3 (GND)
- net at U5.2 (A): now also R20.2
- net COB_LED: now reaches U5.4 (Y)
- net COB_LED: now also J3.2 (Pin_2)
- net 5V: now reaches U5.5 (VCC)
- net 5V: now also C39.1, C40.1.1, J3.3 (Pin_3), J5.3 (Pin_3), U6.5 (VCC)
- new net: R21.2, U6.2 (A)
- new net 3V3: J2.1 (Pin_1), J4.4 (Pin_4)
- new net BTN: J2.5 (Pin_5)
- new net COB_LED_DATA: R20.1
- new net PDM_CLK: J4.2 (Pin_2)
- new net PDM_DATA: J4.3 (Pin_3)
- new net POT1_ADC: J2.3 (Pin_3)
- new net POT2_ADC: J2.4 (Pin_4)
- new net SPK_N: J6.1 (Pin_1)
- new net SPK_P: J6.2 (Pin_2)
- new net WS_LED: J5.2 (Pin_2), U6.4 (Y)
- new net WS_LED_DATA: R21.1
Other:
- note added: "COB LED"
- note added: "Controls Daughterboard"
- note added: "PDM Microphone"
- note added: "Speaker"
- note added: "WS LED"
- moved on the sheet: U5
