File: ESP32-S3_Audio_Control_Board_0707/ESP32-S3_Audio_Control_Board.kicad_pcb (KiCad board)
At the start: 2 copper layers, 60 x 80 mm, 114 parts, among them J1 Barrel_Jack, J10 B5B-PH-K-S(LF)(SN), J2 B2B-PH-K-S(LF)(SN), J3 B4B-PH-K-S(LF)(SN), J5 B3B-PH-K-S(LF)(SN), J9 B3B-PH-K-S(LF)(SN), Q1 AO3401A, U1 ESP32-S3-WROOM-1, U2 TPS54331D, U3 TPS54331D, U4 TAS5805MPWPR, U5 SN74AHCT1G125DBVR, U6 SN74AHCT1G125DBVR

Commit message: update TAS5805, 4-layer
Connections:
- U4 pad 17: unconnected-(U4-OUT_B+-Pad17) -> Net-(U4-OUT_A+)
- U4 pad 20: unconnected-(U4-OUT_B--Pad20) -> Net-(U4-OUT_A-)
Other:
- copper layers 2 -> 4
Changed lines of the file:
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@@
 	(layers
 		(0 "F.Cu" signal)
+		(4 "In1.Cu" signal)
+		(6 "In2.Cu" signal)
 		(2 "B.Cu" signal)
 		(9 "F.Adhes" user "F.Adhesive")
@@
 	)
 	(setup
+		(stackup
+			(layer "F.SilkS"
+				(type "Top Silk Screen")
+			)
+			(layer "F.Paste"
+				(type "Top Solder Paste")
+			)
+			(layer "F.Mask"
+				(type "Top Solder Mask")
+				(thickness 0.01)
+			)
+			(layer "F.Cu"
+				(type "copper")
+				(thickness 0.035)
+			)
+			(layer "dielectric 1"
+				(type "prepreg")
+				(thickness 0.1)
+				(material "FR4")
+				(epsilon_r 4.5)
+				(loss_tangent 0.02)
+			)
+			(layer "In1.Cu"
+				(type "copper")
+				(thickness 0.035)
+			)
+			(layer "dielectric 2"
+				(type "core")
+				(thickness 1.24)
+				(material "FR4")
+				(epsilon_r 4.5)
+				(loss_tangent 0.02)
+			)
+			(layer "In2.Cu"
+				(type "copper")
+				(thickness 0.035)
+			)
+			(layer "dielectric 3"
+				(type "prepreg")
+				(thickness 0.1)
+				(material "FR4")
+				(epsilon_r 4.5)
+				(loss_tangent 0.02)
+			)
+			(layer "B.Cu"
+				(type "copper")
+				(thickness 0.035)
+			)
+			(layer "B.Mask"
+				(type "Bottom Solder Mask")
+				(thickness 0.01)
+			)
+			(layer "B.Paste"
+				(type "Bottom Solder Paste")
+			)
+			(layer "B.SilkS"
+				(type "Bottom Silk Screen")
+			)
+			(copper_finish "None")
+			(dielectric_constraints no)
+		)
 		(pad_to_mask_clearance 0)
 		(allow_soldermask_bridges_in_footprints no)
@@
 		(capping no)
 		(filling no)
+		(zone_defaults)
 		(grid_origin 108 122)
 		(pcbplotparams
@@
 			(layers "F.Cu" "F.Mask" "F.Paste")
 			(roundrect_rratio 0.25)
-			(net "unconnected-(U4-OUT_B+-Pad17)")
+			(net "Net-(U4-OUT_A+)")
 			(pinfunction "OUT_B+_17")
-			(pintype "output+no_connect")
+			(pintype "output")
 		)
 		(pad "18" smd roundrect
@@
 			(layers "F.Cu" "F.Mask" "F.Paste")
 			(roundrect_rratio 0.25)
-			(net "unconnected-(U4-OUT_B--Pad20)")
+			(net "Net-(U4-OUT_A-)")
 			(pinfunction "OUT_B-_20")
-			(pintype "output+no_connect")
+			(pintype "output")
 		)
 		(pad "21" smd roundrect
@@
 		(embedded_fonts no)
 	)
+	(gr_poly
+		(pts
+			(xy 102.793 43.133) (xy 102.793 128.223) (xy 171.754 128.223) (xy 171.754 42.879)
+		)
+		(stroke
+			(width 0.1)
+			(type solid)
+		)
+		(fill yes)
+		(layer "In1.Cu")
+		(net "GND")
+	)
 	(gr_arc
 		(start 105 48)
@@
 	)
 	(group ""
-		(members "00d88eb0-e1f6-4b13-8b11-a23b679cacc7" "0ded1eda-a0d4-489c-97c6-3015749fa674"
-			"115302cd-37cd-4fde-b4e1-f300c2ae2c62" "1898bf03-b3a3-4a75-8d3c-e41a3dbc4cdc"
-			"31efcc32-dabd-45f4-898a-3b67a83c9bb4" "34dbc785-abc8-4318-a094-8d98b9fa4326"
-			"55d84040-663a-4604-834f-19916e08ca1c" "582f0c2b-6a96-4175-a5d7-cd5474a529aa"
-			"61f1f00e-c430-4039-9ac5-905149d2542e" "a5c1b879-94a5-4da8-8c83-f0a4981308b0"
-			"a62b55ba-af1b-4746-9fc2-8195119f43e0" "b3d66ff6-49d1-441d-b7d8-fb6a6952bf04"
-			"b9c349a7-2e8b-4441-a545-026a2b62885e" "ca00dd06-4f4b-4aee-97c8-024ff30c29fa"
-			"d4dbcaa8-b698-4541-acc2-dfba7bdf4c7c" "e6f00886-2626-44e8-b38b-c91e395e8280"
-			"f93978cb-a2e3-40cb-8b77-958b7f3c9fce"
+		(members "0ded1eda-a0d4-489c-97c6-3015749fa674" "115302cd-37cd-4fde-b4e1-f300c2ae2c62"
+			"1898bf03-b3a3-4a75-8d3c-e41a3dbc4cdc" "31efcc32-dabd-45f4-898a-3b67a83c9bb4"
+			"34dbc785-abc8-4318-a094-8d98b9fa4326" "55d84040-663a-4604-834f-19916e08ca1c"
+			"582f0c2b-6a96-4175-a5d7-cd5474a529aa" "61f1f00e-c430-4039-9ac5-905149d2542e"
+			"a5c1b879-94a5-4da8-8c83-f0a4981308b0" "a62b55ba-af1b-4746-9fc2-8195119f43e0"
+			"b3d66ff6-49d1-441d-b7d8-fb6a6952bf04" "b9c349a7-2e8b-4441-a545-026a2b62885e"
+			"ca00dd06-4f4b-4aee-97c8-024ff30c29fa" "d4dbcaa8-b698-4541-acc2-dfba7bdf4c7c"
+			"e6f00886-2626-44e8-b38b-c91e395e8280" "f93978cb-a2e3-40cb-8b77-958b7f3c9fce"
 		)
 	)
@@
 			"07650353-50f4-4f20-a71d-3f45cced4392" "18cfe80a-dcd1-4366-b186-e4f3a02325cf"
 			"1a8b495d-ce6e-48ab-b53f-cd34bd0f8bb2" "20fb8acf-f797-480b-bbf3-d56263e255db"
-			"2ab8e20b-cc5e-4fc7-940e-224b08957e64" "2b4fb054-8fbb-4979-80c1-000776c0c8e5"
-			"3dec1fb9-8e35-41e0-bd4d-1d0aae0ad9b0" "629f6f2c-1b22-48e9-ac15-90c3684fb77e"
-			"67c3de78-0165-47ff-8b31-133f5d8615a9" "79a3d902-cda7-4d6c-a6e5-763244437ed5"
-			"94747d17-1747-4af1-9d3c-11bbd957d68d" "95682246-4131-4f9a-9914-0a33d6458079"
-			"9b60d489-24ef-45c4-bf78-e0fdda73943c" "d3dcdf02-b33f-4363-a913-d64256309ab6"
-			"ddc673a3-64c6-4383-8c38-93c7e6a92589"
+			"2b4fb054-8fbb-4979-80c1-000776c0c8e5" "3dec1fb9-8e35-41e0-bd4d-1d0aae0ad9b0"
+			"629f6f2c-1b22-48e9-ac15-90c3684fb77e" "67c3de78-0165-47ff-8b31-133f5d8615a9"
+			"79a3d902-cda7-4d6c-a6e5-763244437ed5" "94747d17-1747-4af1-9d3c-11bbd957d68d"
+			"95682246-4131-4f9a-9914-0a33d6458079" "9b60d489-24ef-45c4-bf78-e0fdda73943c"
+			"d3dcdf02-b33f-4363-a913-d64256309ab6" "ddc673a3-64c6-4383-8c38-93c7e6a92589"
 		)
 	)
