File: ESP32-S3_Audio_Control_Board_0709/Peri.kicad_sch (KiCad schematic)
At the start: 12 parts, among them J10 B5B-PH-K-S(LF)(SN), J2 B2B-PH-K-S(LF)(SN), J3 B4B-PH-K-S(LF)(SN), J5 B3B-PH-K-S(LF)(SN), J9 B3B-PH-K-S(LF)(SN), U5 SN74AHCT1G125DBVR, U6 SN74AHCT1G125DBVR

Commit message: update
Parts:
- U5, U6: footprint Audio_control_board:SOT95P280X145-5N__SN74AHCT1G125 -> Package_TO_SOT_SMD:SOT-23-5
Connections:
- net COB_LED: now also J5.2 (Pin_2), R20.2; no longer R20.1, U5.4 (Y)
- net WS_LED: now also J9.2 (Pin_2), R21.2; no longer R21.1, U6.4 (Y)
- new net: R21.1, U6.4 (Y)
- new net: R20.1, U5.4 (Y)
Other:
- moved on the sheet: R20, R21
