File: ESP32-S3_Audio_Control_Board_0709/Audio.kicad_sch (KiCad schematic)
At the start: 22 parts, among them U4 TAS5805MPWPR

Commit message: final
Parts:
- C27, C29: Part Description -55℃~+105℃ 10.5mm 2000hrs 25V 3.1mm 390uF 8mm ±20% SMD,D8xL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 -> CAP ALUM POLY 390uF ±20% 25V SMD; Supplier C5246545 -> LCSC; Supplier PN C46550405 -> C5246545
- C34, C36: Mfr Murata Electronics -> YAGEO; Mfr PN GCM31MR71H684KA55L -> CC1206KKX7R9BB684; Part Description 50V 680nF X7R ±10% 1206 Multilayer Ceramic Capacitors MLCC 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 -> CAP CER 680nF 50V X7R 1206; Supplier PN C668325 -> C145012
- R18: Mfr UNI-ROYAL(Uniroyal Elec) -> YAGEO; Mfr PN 0402WGF1002TCE -> RC0402FR-0710KL; Part Description -55℃~+155℃ 10kΩ 50V 62.5mW Thick Film Resistor ±1% ±100ppm/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 -> RES 10kΩ ±1% 62.5mW 0402; Supplier PN C25744 -> C60490
Changed lines of the file:
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@@
 			)
 		)
-		(property "Part Description" "-55℃~+105℃ 10.5mm 2000hrs 25V 3.1mm 390uF 8mm ±20% SMD,D8xL10.5mm Polymer Aluminum Capacitors ROHS"
+		(property "Part Description" "CAP ALUM POLY 390uF ±20% 25V SMD"
 			(at 194.31 52.07 0)
 			(hide yes)
@@
 			)
 		)
-		(property "Supplier" "C5246545"
+		(property "Supplier" "LCSC"
 			(at 194.31 52.07 0)
 			(hide yes)
@@
 			)
 		)
-		(property "Supplier PN" "C46550405"
+		(property "Supplier PN" "C5246545"
 			(at 194.31 52.07 0)
 			(hide yes)
@@
 			)
 		)
-		(property "Part Description" "-55℃~+105℃ 10.5mm 2000hrs 25V 3.1mm 390uF 8mm ±20% SMD,D8xL10.5mm Polymer Aluminum Capacitors ROHS"
+		(property "Part Description" "CAP ALUM POLY 390uF ±20% 25V SMD"
 			(at 143.51 52.07 0)
 			(hide yes)
@@
 			)
 		)
-		(property "Supplier" "C5246545"
+		(property "Supplier" "LCSC"
 			(at 143.51 52.07 0)
 			(hide yes)
@@
 			)
 		)
-		(property "Supplier PN" "C46550405"
+		(property "Supplier PN" "C5246545"
 			(at 143.51 52.07 0)
 			(hide yes)
@@
 			)
 		)
-		(property "Mfr" "Murata Electronics"
+		(property "Mfr" "YAGEO"
 			(at 182.88 82.55 0)
 			(hide yes)
@@
 			)
 		)
-		(property "Mfr PN" "GCM31MR71H684KA55L"
+		(property "Mfr PN" "CC1206KKX7R9BB684"
 			(at 182.88 82.55 0)
 			(hide yes)
@@
 			)
 		)
-		(property "Supplier PN" "C668325"
+		(property "Supplier PN" "C145012"
 			(at 182.88 82.55 0)
 			(hide yes)
@@
 			)
 		)
-		(property "Part Description" "50V 680nF X7R ±10% 1206 Multilayer Ceramic Capacitors MLCC - SMD/SMT ROHS"
+		(property "Part Description" "CAP CER 680nF 50V X7R 1206"
 			(at 182.88 82.55 0)
 			(hide yes)
@@
 			)
 		)
-		(property "Mfr" "UNI-ROYAL(Uniroyal Elec)"
+		(property "Mfr" "YAGEO"
 			(at 101.6 77.47 0)
 			(hide yes)
@@
 			)
 		)
-		(property "Mfr PN" "0402WGF1002TCE"
+		(property "Mfr PN" "RC0402FR-0710KL"
 			(at 101.6 77.47 0)
 			(hide yes)
@@
 			)
 		)
-		(property "Supplier PN" "C25744"
+		(property "Supplier PN" "C60490"
 			(at 101.6 77.47 0)
 			(hide yes)
@@
 			)
 		)
-		(property "Part Description" "-55℃~+155℃ 10kΩ 50V 62.5mW Thick Film Resistor ±1% ±100ppm/℃ 0402 Chip Resistor - Surface Mount ROHS"
+		(property "Part Description" "RES 10kΩ ±1% 62.5mW 0402"
 			(at 101.6 77.47 0)
 			(hide yes)
@@
 			)
 		)
-		(property "Mfr" "Murata Electronics"
+		(property "Mfr" "YAGEO"
 			(at 182.88 97.79 0)
 			(hide yes)
@@
 			)
 		)
-		(property "Mfr PN" "GCM31MR71H684KA55L"
+		(property "Mfr PN" "CC1206KKX7R9BB684"
 			(at 182.88 97.79 0)
 			(hide yes)
@@
 			)
 		)
-		(property "Supplier PN" "C668325"
+		(property "Supplier PN" "C145012"
 			(at 182.88 97.79 0)
 			(hide yes)
@@
 			)
 		)
-		(property "Part Description" "50V 680nF X7R ±10% 1206 Multilayer Ceramic Capacitors MLCC - SMD/SMT ROHS"
+		(property "Part Description" "CAP CER 680nF 50V X7R 1206"
 			(at 182.88 97.79 0)
 			(hide yes)
