File: ESP32-S3_Audio_Control_Board_0709/ESP32-S3.kicad_sch (KiCad schematic)
At the start: 27 parts, among them U1 ESP32-S3-WROOM-1

Commit message: update
Other:
- note added: "USB"
- moved on the sheet: TP11, TP16, TP17

Commit message: update PCB
Connections:
- net USB_DM renamed USB_D_N
- net USB_DP renamed USB_D_P
Changed lines of the file:
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@@
 	(wire
 		(pts
-			(xy 167.64 97.79) (xy 179.07 97.79)
+			(xy 167.64 97.79) (xy 185.42 97.79)
 		)
 		(stroke
@@
 	(wire
 		(pts
-			(xy 167.64 95.25) (xy 179.07 95.25)
+			(xy 167.64 95.25) (xy 185.42 95.25)
 		)
 		(stroke
@@
 		)
 	)
-	(label "USB_DP"
+	(label "USB_D_P"
 		(at 271.78 77.47 180)
 		(effects
@@
 		)
 	)
-	(label "USB_DM"
+	(label "USB_D_N"
 		(at 179.07 95.25 180)
 		(effects
@@
 		)
 	)
-	(label "USB_DP"
+	(label "USB_D_P"
 		(at 179.07 97.79 180)
 		(effects
@@
 		)
 	)
-	(label "USB_DM"
+	(label "USB_D_N"
 		(at 271.78 69.85 180)
 		(effects

Commit message: final
Parts:
- R2, R4: Mfr UNI-ROYAL(Uniroyal Elec) -> YAGEO; Mfr PN 0402WGF1002TCE -> RC0402FR-0710KL; Part Description -55℃~+155℃ 10kΩ 50V 62.5mW Thick Film Resistor ±1% ±100ppm/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 -> RES 10kΩ ±1% 62.5mW 0402; Supplier PN C25744 -> C60490
Changed lines of the file:
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@@
 	)
 	(label "USB_D_N"
-		(at 179.07 95.25 180)
+		(at 185.42 95.25 180)
 		(effects
 			(font
@@
 	)
 	(label "USB_D_P"
-		(at 179.07 97.79 180)
+		(at 185.42 97.79 180)
 		(effects
 			(font
@@
 			)
 		)
-		(property "Mfr" "UNI-ROYAL(Uniroyal Elec)"
+		(property "Mfr" "YAGEO"
 			(at 91.44 119.38 0)
 			(hide yes)
@@
 			)
 		)
-		(property "Mfr PN" "0402WGF1002TCE"
+		(property "Mfr PN" "RC0402FR-0710KL"
 			(at 91.44 119.38 0)
 			(hide yes)
@@
 			)
 		)
-		(property "Supplier PN" "C25744"
+		(property "Supplier PN" "C60490"
 			(at 91.44 119.38 0)
 			(hide yes)
@@
 			)
 		)
-		(property "Part Description" "-55℃~+155℃ 10kΩ 50V 62.5mW Thick Film Resistor ±1% ±100ppm/℃ 0402 Chip Resistor - Surface Mount ROHS"
+		(property "Part Description" "RES 10kΩ ±1% 62.5mW 0402"
 			(at 91.44 119.38 0)
 			(hide yes)
@@
 			)
 		)
-		(property "Mfr" "UNI-ROYAL(Uniroyal Elec)"
+		(property "Mfr" "YAGEO"
 			(at 91.44 80.01 0)
 			(hide yes)
@@
 			)
 		)
-		(property "Mfr PN" "0402WGF1002TCE"
+		(property "Mfr PN" "RC0402FR-0710KL"
 			(at 91.44 80.01 0)
 			(hide yes)
@@
 			)
 		)
-		(property "Supplier PN" "C25744"
+		(property "Supplier PN" "C60490"
 			(at 91.44 80.01 0)
 			(hide yes)
@@
 			)
 		)
-		(property "Part Description" "-55℃~+155℃ 10kΩ 50V 62.5mW Thick Film Resistor ±1% ±100ppm/℃ 0402 Chip Resistor - Surface Mount ROHS"
+		(property "Part Description" "RES 10kΩ ±1% 62.5mW 0402"
 			(at 91.44 80.01 0)
 			(hide yes)
