File: ESP32-S3_Audio_Control_Board_0709/ESP32-S3_Audio_Control_Board.kicad_pcb (KiCad board)
At the start: 4 copper layers, 60 x 80 mm, 116 parts, among them J1 Barrel_Jack, J10 B5B-PH-K-S(LF)(SN), J2 B2B-PH-K-S(LF)(SN), J3 B4B-PH-K-S(LF)(SN), J5 B3B-PH-K-S(LF)(SN), J9 B3B-PH-K-S(LF)(SN), U1 ESP32-S3-WROOM-1, U2 TPS54331D, U3 TPS54331D, U4 TAS5805MPWPR, U5 SN74AHCT1G125DBVR, U6 SN74AHCT1G125DBVR

Commit message: update
Parts:
- J1: value Barrel_Jack -> PJ-102AH
- U5, U6: footprint Audio_control_board:SOT95P280X145-5N__SN74AHCT1G125 -> Package_TO_SOT_SMD:SOT-23-5
- moved TP16 11.4 mm to (135.8, 82.0)
- moved TP17 7.71 mm to (135.8, 79.5)
- moved R20 2.69 mm to (142.5, 61.9)
- moved C40 2.43 mm to (143.6, 104.2)
- moved U6 2.43 mm to (141.1, 104.2)
- moved C39 2.29 mm to (139.2, 65.5)
- moved U5 2.29 mm to (141.5, 65.5)
- moved R21 1.92 mm to (140.1, 107.6)
Connections:
- J5 pad 2: Net-(J5-Pin_2) -> /Peripheral/COB_LED
- J9 pad 2: Net-(J9-Pin_2) -> /Peripheral/WS_LED
- R20 pad 1: /Peripheral/COB_LED -> Net-(U5-Y)
- R20 pad 2: Net-(J5-Pin_2) -> /Peripheral/COB_LED
- R21 pad 1: /Peripheral/WS_LED -> Net-(U6-Y)
- R21 pad 2: Net-(J9-Pin_2) -> /Peripheral/WS_LED
- U5 pad 4: /Peripheral/COB_LED -> Net-(U5-Y)
- U6 pad 4: /Peripheral/WS_LED -> Net-(U6-Y)
Other:
- board text added: "BOTTOM LAYER"
- board text added: "LAYER 2(GND)"
- board text added: "LAYER 3(PWR)"
- board text added: "TOP LAYER"

Commit message: update PCB
Parts:
- removed the R20 at (152.3, 73.0)
- removed the R21 at (145.8, 97.2)
- removed TP3: IO0, TestPoint:TestPoint_Pad_D1.5mm
- moved D2 19.8 mm to (111.6, 62.5), turned to 90 degrees
- moved C14 2.12 mm to (108.6, 64.0), turned to 90 degrees
- moved C41 2.03 mm to (106.7, 63.5), turned to 90 degrees
- moved J1 1.78 mm to (119.9, 59.0)
- moved R16 1.67 mm to (131.9, 70.9), turned to 180 degrees
- moved R4 1.52 mm to (140.8, 95.7)
- moved C34 1.32 mm to (112.4, 111.3)
- moved C2 1.31 mm to (156.5, 73.7)
- moved C1 1.29 mm to (156.8, 72.5)
- moved TP14 1.27 mm to (150.5, 69.2)
- moved TP15 1.27 mm to (150.5, 65.9)
- moved C28 1.21 mm to (127.5, 112.5)
- moved C44 1.21 mm to (127.5, 114.9)
- moved R11 1.19 mm to (111.4, 83.5), turned to 90 degrees
- moved C3 1.18 mm to (156.5, 74.8)
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Connections:
- net /ESP32-S3/USB_DM renamed /ESP32-S3/USB_D_N
- net /ESP32-S3/USB_DP renamed /ESP32-S3/USB_D_P
Routing:
- net 3V3: track 0.00 -> 171.0 mm, vias 0 -> 8
- net 5V: track 0.00 -> 95.8 mm, vias 0 -> 5
- net 12V: track 0.00 -> 61.1 mm, vias 0 -> 10
- net BCLK: track 0.00 -> 60.4 mm, vias 0 -> 1
- net LRCLK: track 0.00 -> 57.7 mm
- net DOUT: track 0.00 -> 56.9 mm, vias 0 -> 2
- net PVDD: track 0.00 -> 48.4 mm, vias 0 -> 2
- net BTN: track 0.00 -> 44.2 mm, vias 0 -> 2
- net AMP_FAULTZ: track 0.00 -> 43.1 mm, vias 0 -> 2
- net /ESP32-S3/EN: track 0.00 -> 41.0 mm, vias 0 -> 1
- net PDM_DATA: track 0.00 -> 36.8 mm, vias 0 -> 3
- net /ESP32-S3/TXD: track 0.00 -> 35.7 mm, vias 0 -> 1
- net /ESP32-S3/RXD: track 0.00 -> 30.4 mm, vias 0 -> 1
- net PDM_CLK: track 0.00 -> 26.0 mm, vias 0 -> 2
- net Net-(U4-OUT_A+): track 0.00 -> 23.2 mm
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- added copper zone on F.Cu, net 12V
- added copper zone on In2.Cu, net 12V
- added copper zone on F.Cu, net 3V3
- added copper zone on In2.Cu, net 3V3
- added copper zone on F.Cu, net 5V
- added copper zone on In2.Cu, net 5V
- added copper zone on B.Cu, net GND
- added copper zone on F.Cu, net GND
- added copper zone on In1.Cu, net GND
- added copper zone on In2.Cu, net GND
- added copper zone on In2.Cu, net Net-(C13-Pad1)
- added copper zone on F.Cu, net Net-(D1-K)
- added copper zone on F.Cu, net Net-(D3-K)
- added copper zone on F.Cu, net PVDD
- added copper zone on In2.Cu, net PVDD

Commit message: update
Parts:
- moved J2 0.25 mm to (107.3, 107.3)
Routing:
- net 3V3: vias 8 -> 9
- net GND: vias 66 -> 95
- added copper zone on F.Cu, net Net-(C13-Pad1)

Commit message: final
Parts:
- added TP3: IO0, TestPoint:TestPoint_Pad_D1.5mm, B.Cu at (132.0, 82.0)
- moved L2 0.38 mm to (133.6, 65.7)
- moved C1 0.15 mm to (156.8, 72.3)
- moved L1 0.15 mm to (116.8, 84.8)
- moved TP16 0.13 mm to (136.7, 82.0)
- moved TP17 0.13 mm to (136.7, 79.5)
Routing:
- net 3V3: track 171.0 -> 39.1 mm, vias 9 -> 12
- net 5V: track 95.8 -> 9.20 mm, vias 5 -> 16
- net PVDD: track 48.4 -> 0.00 mm, vias 2 -> 12
- net 12V: track 61.1 -> 23.9 mm, vias 10 -> 16
- net Net-(C13-Pad1): track 7.01 -> 1.45 mm, vias 1 -> 7
- net Net-(U4-OUT_A-): track 12.6 -> 8.25 mm
- net SPK_P: track 9.05 -> 6.18 mm
- net SPK_N: track 9.05 -> 6.18 mm
- net /ESP32-S3/USB_D_N: track 18.0 -> 18.5 mm
- net GND: vias 95 -> 205
- added copper zone on F.Cu, net Net-(U4-OUT_A+)
- added copper zone on F.Cu, net Net-(U4-OUT_A-)
- added copper zone on F.Cu, net SPK_N
- added copper zone on F.Cu, net SPK_P
Other:
- board text added: "3V3"
- board text added: "5V"
- board text added: "BCLK"
- board text added: "EN"
- board text added: "GND"
- board text added: "IO0"
- board text added: "LED_COB"
- board text added: "PDM_DATA"
- board text added: "RXD"
- board text added: "TXD"
- board text added: "USB_DN"
- board text added: "USB_DP"
