File: ESP32-S3_Audio_Control_Board_0709/PWR.kicad_sch (KiCad schematic)
At the start: 43 parts, among them J1 Barrel_Jack, U2 TPS54331D, U3 TPS54331D

Commit message: update
Parts:
- D2: Mfr (none) -> Littelfuse; Mfr PN (none) -> SMAJ13A; Part Description (none) -> TVS DIODE 13VWM 21.5VC DO-214AC(SMA); Supplier (none) -> LCSC; Supplier PN (none) -> C148214
- J1: value Barrel_Jack -> PJ-102AH; Part Description DC Power Connectors PCB 2.1MM -> CONN PWR JACK 2mm x 6.5mm

Commit message: final
Parts:
- C19, C42, C43, C9: Mfr Murata Electronics -> YAGEO; Mfr PN GRM1555CYA103JE01D -> CC0402KRX7R9BB103; Part Description 10nF 35V C0G ±5% 0402 Multilayer Ceramic Capacitors MLCC - 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 -> CAP CER 10nF 50V X7R 0402; Supplier PN C1518210 -> C60133
Changed lines of the file:
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@@
 			)
 		)
-		(property "Description" "10nF 35V C0G ±5% 0402"
+		(property "Description" ""
 			(at 60.96 129.54 0)
 			(hide yes)
@@
 			)
 		)
-		(property "Mfr" "Murata Electronics"
+		(property "Mfr" "YAGEO"
 			(at 60.96 129.54 0)
 			(hide yes)
@@
 			)
 		)
-		(property "Mfr PN" "GRM1555CYA103JE01D"
+		(property "Mfr PN" "CC0402KRX7R9BB103"
 			(at 60.96 129.54 0)
 			(hide yes)
@@
 			)
 		)
-		(property "Supplier PN" "C1518210"
+		(property "Supplier PN" "C60133"
 			(at 60.96 129.54 0)
 			(hide yes)
@@
 			)
 		)
-		(property "Part Description" "10nF 35V C0G ±5% 0402 Multilayer Ceramic Capacitors MLCC - SMD/SMT ROHS "
+		(property "Part Description" "CAP CER 10nF 50V X7R 0402"
 			(at 60.96 129.54 0)
 			(hide yes)
@@
 			)
 		)
-		(property "Description" "10nF 35V C0G ±5% 0402"
+		(property "Description" ""
 			(at 181.61 128.27 0)
 			(hide yes)
@@
 			)
 		)
-		(property "Mfr" "Murata Electronics"
+		(property "Mfr" "YAGEO"
 			(at 181.61 128.27 0)
 			(hide yes)
@@
 			)
 		)
-		(property "Mfr PN" "GRM1555CYA103JE01D"
+		(property "Mfr PN" "CC0402KRX7R9BB103"
 			(at 181.61 128.27 0)
 			(hide yes)
@@
 			)
 		)
-		(property "Supplier PN" "C1518210"
+		(property "Supplier PN" "C60133"
 			(at 181.61 128.27 0)
 			(hide yes)
@@
 			)
 		)
-		(property "Part Description" "10nF 35V C0G ±5% 0402 Multilayer Ceramic Capacitors MLCC - SMD/SMT ROHS "
+		(property "Part Description" "CAP CER 10nF 50V X7R 0402"
 			(at 181.61 128.27 0)
 			(hide yes)
@@
 			)
 		)
-		(property "Description" "10nF 35V C0G ±5% 0402"
+		(property "Description" ""
 			(at 193.04 83.82 0)
 			(hide yes)
@@
 			)
 		)
-		(property "Mfr" "Murata Electronics"
+		(property "Mfr" "YAGEO"
 			(at 193.04 83.82 0)
 			(hide yes)
@@
 			)
 		)
-		(property "Mfr PN" "GRM1555CYA103JE01D"
+		(property "Mfr PN" "CC0402KRX7R9BB103"
 			(at 193.04 83.82 0)
 			(hide yes)
@@
 			)
 		)
-		(property "Supplier PN" "C1518210"
+		(property "Supplier PN" "C60133"
 			(at 193.04 83.82 0)
 			(hide yes)
@@
 			)
 		)
-		(property "Part Description" "10nF 35V C0G ±5% 0402 Multilayer Ceramic Capacitors MLCC - SMD/SMT ROHS "
+		(property "Part Description" "CAP CER 10nF 50V X7R 0402"
 			(at 193.04 83.82 0)
 			(hide yes)
@@
 			)
 		)
-		(property "Description" "10nF 35V C0G ±5% 0402"
+		(property "Description" ""
 			(at 72.39 83.82 0)
 			(hide yes)
@@
 			)
 		)
-		(property "Mfr" "Murata Electronics"
+		(property "Mfr" "YAGEO"
 			(at 72.39 83.82 0)
 			(hide yes)
@@
 			)
 		)
-		(property "Mfr PN" "GRM1555CYA103JE01D"
+		(property "Mfr PN" "CC0402KRX7R9BB103"
 			(at 72.39 83.82 0)
 			(hide yes)
@@
 			)
 		)
-		(property "Supplier PN" "C1518210"
+		(property "Supplier PN" "C60133"
 			(at 72.39 83.82 0)
 			(hide yes)
@@
 			)
 		)
-		(property "Part Description" "10nF 35V C0G ±5% 0402 Multilayer Ceramic Capacitors MLCC - SMD/SMT ROHS "
+		(property "Part Description" "CAP CER 10nF 50V X7R 0402"
 			(at 72.39 83.82 0)
 			(hide yes)
